File: keyboard-layout-tall/keyboard-layout-tall.kicad_pcb (KiCad board)
At the start: 2 copper layers, 308 x 143 mm, 176 parts, among them J1 Conn_01x26, J2 Conn_01x04, K0 KEYSW, K1 KEYSW, K10 KEYSW, K11 KEYSW, K12 KEYSW, K13 KEYSW, K14 KEYSW, K15 KEYSW, K16 KEYSW, K17 KEYSW, K18 KEYSW, K19 KEYSW, K2 KEYSW, K20 KEYSW, K21 KEYSW, K22 KEYSW, K23 KEYSW, K24 KEYSW, K25 KEYSW, K26 KEYSW, K27 KEYSW, K28 KEYSW, K29 KEYSW, K3 KEYSW, K30 KEYSW, K31 KEYSW, K32 KEYSW, K33 KEYSW, K34 KEYSW, K35 KEYSW, K36 KEYSW, K37 KEYSW, K38 KEYSW, K39 KEYSW, K4 KEYSW, K40 KEYSW, K41 KEYSW, K42 KEYSW, K43 KEYSW, K44 KEYSW, K45 KEYSW, K46 KEYSW, K47 KEYSW, K48 KEYSW, K49 KEYSW, K5 KEYSW, K50 KEYSW, K51 KEYSW, K52 KEYSW, K53 KEYSW, K54 KEYSW, K55 KEYSW, K56 KEYSW, K57 KEYSW, K58 KEYSW, K59 KEYSW, K6 KEYSW, K60 KEYSW, K61 KEYSW, K62 KEYSW, K63 KEYSW, K64 KEYSW, K65 KEYSW, K66 KEYSW, K67 KEYSW, K68 KEYSW, K69 KEYSW, K7 KEYSW, K70 KEYSW, K71 KEYSW, K72 KEYSW, K73 KEYSW, K74 KEYSW, K75 KEYSW, K76 KEYSW, K77 KEYSW, K8 KEYSW, K9 KEYSW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

Commit message: Updated board to remove diodes. 2021-05-15 version should work right out of the box.
Parts:
- removed D0, D1, D10, D11, D12, D13, D14, D15, D16, D17, D18, D19, D2, D20, D21, D22, D23, D24, D25, D26, D27, D28, D29, D3, D30, D31, D32, D33, D34, D35, D36, D37, D38, D39, D4, D40, D41, D42, D43, D44, D45, D46, D47, D48, D49, D5, D50, D51, D52, D53, D54, D55, D56, D57, D58, D59, D6, D60, D61, D62, D63, D64, D65, D66, D67, D68, D69, D7, D70, D71, D72, D73, D74, D75, D76, D77, D8, D9: D, Diode_SMD:D_SOD-123F
Connections:
- K0 pad 2: Net-(D0-Pad2) -> /Row_4
- K1 pad 2: Net-(D1-Pad2) -> /Row_1
- K10 pad 2: Net-(D10-Pad2) -> /Row_0
- K11 pad 2: Net-(D11-Pad2) -> /Row_1
- K12 pad 2: Net-(D12-Pad2) -> /Row_0
- K13 pad 2: Net-(D13-Pad2) -> /Row_0
- K14 pad 2: Net-(D14-Pad2) -> /Row_0
- K15 pad 2: Net-(D15-Pad2) -> /Row_0
- K16 pad 2: Net-(D16-Pad2) -> /Row_1
- K17 pad 2: Net-(D17-Pad2) -> /Row_1
- K18 pad 2: Net-(D18-Pad2) -> /Row_0
- K19 pad 2: Net-(D19-Pad2) -> /Row_0
- K2 pad 2: Net-(D2-Pad2) -> /Row_1
- K20 pad 2: Net-(D20-Pad2) -> /Row_0
- K21 pad 2: Net-(D21-Pad2) -> /Row_0
- K22 pad 2: Net-(D22-Pad2) -> /Row_1
- K23 pad 2: Net-(D23-Pad2) -> /Row_1
- K24 pad 2: Net-(D24-Pad2) -> /Row_6
- K25 pad 2: Net-(D25-Pad2) -> /Row_3
- K26 pad 2: Net-(D26-Pad2) -> /Row_6
- K27 pad 2: Net-(D27-Pad2) -> /Row_7
- K28 pad 2: Net-(D28-Pad2) -> /Row_7
- K29 pad 2: Net-(D29-Pad2) -> /Row_7
- K3 pad 2: Net-(D3-Pad2) -> /Row_6
- K30 pad 2: Net-(D30-Pad2) -> /Row_7
- K31 pad 2: Net-(D31-Pad2) -> /Row_6
- K32 pad 2: Net-(D32-Pad2) -> /Row_6
- K33 pad 2: Net-(D33-Pad2) -> /Row_7
- K34 pad 2: Net-(D34-Pad2) -> /Row_7
- K35 pad 2: Net-(D35-Pad2) -> /Row_7
- K36 pad 2: Net-(D36-Pad2) -> /Row_7
- K37 pad 2: Net-(D37-Pad2) -> /Row_6
- K38 pad 2: Net-(D38-Pad2) -> /Row_6
- K39 pad 2: Net-(D39-Pad2) -> /Row_5
- K4 pad 2: Net-(D4-Pad2) -> /Row_4
- K40 pad 2: Net-(D40-Pad2) -> /Row_1
- K41 pad 2: Net-(D41-Pad2) -> /Row_6
- K42 pad 2: Net-(D42-Pad2) -> /Row_5
- K43 pad 2: Net-(D43-Pad2) -> /Row_5
- K44 pad 2: Net-(D44-Pad2) -> /Row_5
- K45 pad 2: Net-(D45-Pad2) -> /Row_5
- K46 pad 2: Net-(D46-Pad2) -> /Row_4
- K47 pad 2: Net-(D47-Pad2) -> /Row_4
- K48 pad 2: Net-(D48-Pad2) -> /Row_5
- K49 pad 2: Net-(D49-Pad2) -> /Row_5
- K5 pad 2: Net-(D5-Pad2) -> /Row_0
- K50 pad 2: Net-(D50-Pad2) -> /Row_5
- K51 pad 2: Net-(D51-Pad2) -> /Row_5
- K52 pad 2: Net-(D52-Pad2) -> /Row_4
- K53 pad 2: Net-(D53-Pad2) -> /Row_3
- K54 pad 2: Net-(D54-Pad2) -> /Row_0
- K55 pad 2: Net-(D55-Pad2) -> /Row_5
- K56 pad 2: Net-(D56-Pad2) -> /Row_3
- K57 pad 2: Net-(D57-Pad2) -> /Row_3
- K58 pad 2: Net-(D58-Pad2) -> /Row_3
- K59 pad 2: Net-(D59-Pad2) -> /Row_3
- K6 pad 2: Net-(D6-Pad2) -> /Row_4
- K60 pad 2: Net-(D60-Pad2) -> /Row_2
- K61 pad 2: Net-(D61-Pad2) -> /Row_2
- K62 pad 2: Net-(D62-Pad2) -> /Row_3
- K63 pad 2: Net-(D63-Pad2) -> /Row_3
- K64 pad 2: Net-(D64-Pad2) -> /Row_3
- K65 pad 2: Net-(D65-Pad2) -> /Row_2
- K66 pad 2: Net-(D66-Pad2) -> /Row_6
- K67 pad 2: Net-(D67-Pad2) -> /Row_4
- K68 pad 2: Net-(D68-Pad2) -> /Row_5
- K69 pad 2: Net-(D69-Pad2) -> /Row_1
- K7 pad 2: Net-(D7-Pad2) -> /Row_6
- K70 pad 2: Net-(D70-Pad2) -> /Row_6
- K71 pad 2: Net-(D71-Pad2) -> /Row_4
- K72 pad 2: Net-(D72-Pad2) -> /Row_4
- K73 pad 2: Net-(D73-Pad2) -> /Row_2
- K74 pad 2: Net-(D74-Pad2) -> /Row_3
- K75 pad 2: Net-(D75-Pad2) -> /Row_2
- K76 pad 2: Net-(D76-Pad2) -> /Row_2
- K77 pad 2: Net-(D77-Pad2) -> /Row_2
- K8 pad 2: Net-(D8-Pad2) -> /Row_1
- K9 pad 2: Net-(D9-Pad2) -> /Row_1
Routing:
- net /Row_0: track 374.1 -> 444.3 mm
- net /Row_3: track 482.1 -> 550.8 mm, vias 6 -> 8
- net /Row_6: track 559.8 -> 622.5 mm, vias 7 -> 12
- net /Row_7: track 251.6 -> 309.4 mm
- net /Row_2: track 294.2 -> 344.6 mm, vias 5 -> 9
- net /Row_5: track 453.9 -> 501.4 mm
- net /Row_4: track 607.1 -> 651.0 mm, vias 7 -> 12
- net /Row_1: track 505.8 -> 549.4 mm, vias 6 -> 15
- net Net-(D68-Pad2): track 5.23 -> 0.00 mm
- net Net-(D67-Pad2): track 5.23 -> 0.00 mm
- net Net-(D66-Pad2): track 5.23 -> 0.00 mm
- net Net-(D65-Pad2): track 5.23 -> 0.00 mm
- net Net-(D64-Pad2): track 5.23 -> 0.00 mm
- net Net-(D63-Pad2): track 5.23 -> 0.00 mm
- net Net-(D62-Pad2): track 5.23 -> 0.00 mm
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Other:
- board text added: "Pi 400 Mechanical Keyboard by rglenn 2021-05-15"
- board text removed: "Pi 400 Mechanical Keyboard by rglenn 2021-03-28"
