File: keyboard-layout-tall/keyboard-layout-tall.sch (KiCad schematic (older format))
At the start: 176 parts, among them J1 Conn_01x26, J2 Conn_01x04, K0 KEYSW, K1 KEYSW, K10 KEYSW, K11 KEYSW, K12 KEYSW, K13 KEYSW, K14 KEYSW, K15 KEYSW, K16 KEYSW, K17 KEYSW, K18 KEYSW, K19 KEYSW, K2 KEYSW, K20 KEYSW, K21 KEYSW, K22 KEYSW, K23 KEYSW, K24 KEYSW, K25 KEYSW, K26 KEYSW, K27 KEYSW, K28 KEYSW, K29 KEYSW, K3 KEYSW, K30 KEYSW, K31 KEYSW, K32 KEYSW, K33 KEYSW, K34 KEYSW, K35 KEYSW, K36 KEYSW, K37 KEYSW, K38 KEYSW, K39 KEYSW, K4 KEYSW, K40 KEYSW, K41 KEYSW, K42 KEYSW, K43 KEYSW, K44 KEYSW, K45 KEYSW, K46 KEYSW, K47 KEYSW, K48 KEYSW, K49 KEYSW, K5 KEYSW, K50 KEYSW, K51 KEYSW, K52 KEYSW, K53 KEYSW, K54 KEYSW, K55 KEYSW, K56 KEYSW, K57 KEYSW, K58 KEYSW, K59 KEYSW, K6 KEYSW, K60 KEYSW, K61 KEYSW, K62 KEYSW, K63 KEYSW, K64 KEYSW, K65 KEYSW, K66 KEYSW, K67 KEYSW, K68 KEYSW, K69 KEYSW, K7 KEYSW, K70 KEYSW, K71 KEYSW, K72 KEYSW, K73 KEYSW, K74 KEYSW, K75 KEYSW, K76 KEYSW, K77 KEYSW, K8 KEYSW, K9 KEYSW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

Commit message: Updated board to remove diodes. 2021-05-15 version should work right out of the box.
Parts:
- removed D0, D1, D10, D11, D12, D13, D14, D15, D16, D17, D18, D19, D2, D20, D21, D22, D23, D24, D25, D26, D27, D28, D29, D3, D30, D31, D32, D33, D34, D35, D36, D37, D38, D39, D4, D40, D41, D42, D43, D44, D45, D46, D47, D48, D49, D5, D50, D51, D52, D53, D54, D55, D56, D57, D58, D59, D6, D60, D61, D62, D63, D64, D65, D66, D67, D68, D69, D7, D70, D71, D72, D73, D74, D75, D76, D77, D8, D9: D, Diode_SMD:D_SOD-123F, symbol Device:D
Connections:
- net Row_0: now also K10.2, K12.2, K13.2, K14.2, K15.2, K18.2, K19.2, K20.2, K21.2, K5.2, K54.2
- net Row_1: now also K1.2, K11.2, K16.2, K17.2, K2.2, K22.2, K23.2, K40.2, K69.2, K8.2, K9.2
- net Row_2: now also K60.2, K61.2, K65.2, K73.2, K75.2, K76.2, K77.2
- net Row_3: now also K25.2, K53.2, K56.2, K57.2, K58.2, K59.2, K62.2, K63.2, K64.2, K74.2
- net Row_4: now also K0.2, K4.2, K46.2, K47.2, K52.2, K6.2, K67.2, K71.2, K72.2
- net Row_5: now also K39.2, K42.2, K43.2, K44.2, K45.2, K48.2, K49.2, K50.2, K51.2, K55.2, K68.2
- net Row_6: now also K24.2, K26.2, K3.2, K31.2, K32.2, K37.2, K38.2, K41.2, K66.2, K7.2, K70.2
- net Row_7: now also K27.2, K28.2, K29.2, K30.2, K33.2, K34.2, K35.2, K36.2
